Commit message: feat: added ros2_control xacro

File: urdf/common.gazebo.xacro (robot description, xacro)
@@ -2,6 +2,41 @@
 <robot xmlns:xacro="http://www.ros.org/wiki/xacro">
 	<!-- ROS CONTROL GAZEBO PLUGIN -->
-    <!-- <xacro:macro name="ros2_control">
-	</xacro:macro> -->
+	<xacro:macro name="ros2_control_gazebo">
+		<ros2_control name="gazebo_ros2_control" type="system">
+			<hardware>
+				<plugin>gazebo_ros2_control/GazeboSystem</plugin>
+			</hardware>
+			<joint name="robot_left_wheel_joint">
+				<command_interface name="velocity">
+					<param name="min">-1</param>
+					<param name="max">1</param>
+				</command_interface>
+				<state_interface name="position"/>
+				<state_interface name="velocity"/>
+			</joint>
+			<joint name="robot_right_wheel_joint">
+				<command_interface name="velocity">
+					<param name="min">-1</param>
+					<param name="max">1</param>
+				</command_interface>
+				<state_interface name="position"/>
+				<state_interface name="velocity"/>
+			</joint>
+			<joint name="robot_elevator_platform_joint">
+				<command_interface name="effort">
+					<param name="min">0.0</param>
+					<param name="max">10.0</param>
+				</command_interface>
+				<state_interface name="position"/>
+				<state_interface name="velocity"/>
+				<state_interface name="effort"/>
+			</joint>
+		</ros2_control>
+		<gazebo>
+			<plugin filename="libgazebo_ros2_control.so" name="gazebo_ros2_control">
+				<parameters>$(find rb1_ros2_description)/config/rb1_controller.yaml</parameters>
+			</plugin>
+		</gazebo>
+	</xacro:macro>
 	<xacro:macro name="gazebo_colors" params="prefix">
 		<gazebo reference="$(arg prefix)base_footprint">

File: xacro/rb1_ros2_base.urdf.xacro (robot description, xacro)
@@ -85,4 +85,4 @@
 	</xacro:sensor_orbbec_astra>
 	<!-- Gazebo ros2 control plugins -->
-	<!-- <xacro:ros2_control/> -->
+	<xacro:ros2_control_gazebo/>
 </robot>
